Commit message: Funcionamiento de 2 motores maxon con ros bridge

File: maxon_canopen/urdf/maxon_epos4_1dof_ppm.xacro (robot description, xacro)
@@ -9,18 +9,18 @@
   </link>
   <!-- Joint between Base Link and Link1 Link -->
-  <joint name="base_link1_joint" type="revolute">
+  <joint name="base_link2_joint" type="revolute">
     <parent link="base_link"/>
     <child link="link1_link"/>
     <origin xyz="0 0 0" rpy="0 0 0"/>
     <axis xyz="1 0 0"/>
-    <!--dynamics damping="0.7"/-->
-    <limit effort="100.0" velocity="100000" lower="-100000.0" upper="100000.0"/>
+    <dynamics damping="0.7"/>
+    <limit effort="100.0" velocity="200000" lower="-2654208.0" upper="2654208.0"/>
   </joint>
   <transmission name="transmission_base_link1">
     <type>transmission_interface/SimpleTransmission</type>
-    <joint name="base_link1_joint">
+    <joint name="base_link2_joint">
       <hardwareInterface>hardware_interface/EffortJointInterface</hardwareInterface>
     </joint>
-    <actuator name="link1_maxon_motor">
+    <actuator name="link2_maxon_motor">
       <hardwareInterface>EffortJointInterface</hardwareInterface>
       <mechanicalReduction>1</mechanicalReduction>

File: maxon_canopen/urdf/maxon_epos4_2dof_pvm.xacro (robot description, xacro)
@@ -9,11 +9,11 @@
   </link>
   <!-- Joint between Base link and Link1 link -->
-  <joint name="base_link1_joint" type="continuous">
+  <joint name="base_link1_joint" type="revolute">
     <parent link="base_link"/>
     <child link="link1_link"/>
     <origin xyz="0 0 0" rpy="0 0 0"/>
-    <axis xyz="1 0 0"/>
+    <axis xyz="0 1 0"/>
     <dynamics damping="0.7"/>
-    <limit effort="100.0" velocity="1300"/>
+    <limit effort="100.0" velocity="100000" lower="-4265420.0" upper="465420.0"/>
   </joint>
   <!-- Link2 Link -->
@@ -21,5 +21,5 @@
   </link>
   <!-- Joint between Base link and Link2 link -->
-  <joint name="base_link2_joint" type="continuous">
+  <joint name="base_link2_joint" type="revolute">
     <parent link="base_link"/>
     <child link="link2_link"/>
@@ -27,5 +27,5 @@
     <axis xyz="1 0 0"/>
     <dynamics damping="0.7"/>
-    <limit effort="100.0" velocity="1300"/>
+    <limit effort="100.0" velocity="200000" lower="-2654208.0" upper="2654208.0"/>
   </joint>
   <transmission name="transmission_base_link1">
